Commit message: copy given files

File: ros_ws/install/share/baxter_description/urdf/baxter.urdf.xacro (robot description, xacro)
@@ -1,6 +1,7 @@
 <?xml version="1.0" ?>
 <robot name="baxter" xmlns:xacro="http://www.ros.org/wiki/xacro">
-  <xacro:arg name="gazebo" default="false"/>
+  <xacro:arg name="gazebo" default="true"/>
   <xacro:arg name="pedestal" default="true"/>
+  <xacro:arg name="coffe_table" default="true"/>
   <!-- Baxter Base URDF -->
   <xacro:include filename="$(find baxter_description)/urdf/baxter_base/baxter_base.urdf.xacro">
@@ -17,3 +18,5 @@
   <!-- Right End Effector -->
   <xacro:include filename="$(find baxter_description)/urdf/right_end_effector.urdf.xacro" />
+  <!-- Coffe Table -->
+  <xacro:include filename="$(find baxter_sim_examples)/models/cafe_table/model.xacro" />
 </robot>

File: ros_ws/install/share/baxter_description/urdf/baxter_base/baxter_base.urdf.xacro (robot description, xacro)
@@ -186,10 +186,10 @@
   <joint name="collision_head_1" type="fixed">
     <origin rpy="0 0 0" xyz="0.11 0 0.75"/>
-    <parent link="base"/>
+    <parent link="torso"/>
     <child link="collision_head_link_1"/>
   </joint>
   <joint name="collision_head_2" type="fixed">
     <origin rpy="0 0 0" xyz="0.11 0 0.75"/>
-    <parent link="base"/>
+    <parent link="torso"/>
     <child link="collision_head_link_2"/>
   </joint>
@@ -200,5 +200,5 @@
   </joint>
   <joint name="torso_t0" type="fixed">
-    <origin rpy="0 0 0" xyz="0 0 0"/>
+    <origin rpy="0 0 0" xyz="0 0 0.93"/>
     <parent link="base"/>
     <child link="torso"/>
